File: Cramps2nano-soc/Cramps2_nano-soc.sch (KiCad schematic (older format))
At the start: 6 parts, among them P8 BB_EXP_CONN, P9 BB_EXP_CONN

Commit message: add 3.3 voltage ref resistor on adc ch 8
Signed-off-by: Michael Brown <producer@holotronic.dk>
Parts:
- added R1: 120R, symbol R
- gave numbers to parts that had none: 1
- renumbered ADC to ADC1
Connections:
- net +3V3: now also R1.1
- net at ADC1.9 (P9): now also R1.2
Changed lines of the file:
@@
 DGND
 $Comp
-L PWR_FLAG #FLG?
+L PWR_FLAG #FLG1
 U 1 1 5813F80B
 P 14050 6850
-F 0 "#FLG?" H 14050 6945 30  0001 C CNN
+F 0 "#FLG1" H 14050 6945 30  0001 C CNN
 F 1 "PWR_FLAG" H 14050 7030 30  0000 C CNN
 F 2 "" H 14050 6850 60  0001 C CNN
@@
 $EndComp
 $Comp
-L GND #PWR?
+L GND #PWR1
 U 1 1 5813F80C
 P 14050 6950
-F 0 "#PWR?" H 14050 6950 30  0001 C CNN
+F 0 "#PWR1" H 14050 6950 30  0001 C CNN
 F 1 "GND" H 14050 6880 30  0001 C CNN
 F 2 "" H 14050 6950 60  0001 C CNN
@@
 $EndComp
 $Comp
-L HEADER_6 P?
+L HEADER_6 P1
 U 1 1 5813F818
 P 14250 8550
-F 0 "P?" H 14250 8900 60  0000 C CNN
+F 0 "P1" H 14250 8900 60  0000 C CNN
 F 1 "SOCKET_6_LONG" H 14250 8200 60  0001 C CNN
 F 2 "pin_strip_6" H 14250 8550 60  0001 C CNN
@@
 BeagleBone Logic supply is always 3.3V
 $Comp
-L PWR_FLAG #FLG?
+L PWR_FLAG #FLG2
 U 1 1 5813F819
 P 14300 5900
-F 0 "#FLG?" H 14300 5995 30  0001 C CNN
+F 0 "#FLG2" H 14300 5995 30  0001 C CNN
 F 1 "PWR_FLAG" H 14300 6080 30  0000 C CNN
 F 2 "" H 14300 5900 60  0001 C CNN
@@
 	14100 6400 14100 6300
 $Comp
-L +5V #PWR?
+L +5V #PWR3
 U 1 1 5813F81A
 P 14100 6300
-F 0 "#PWR?" H 14100 6390 20  0001 C CNN
+F 0 "#PWR3" H 14100 6390 20  0001 C CNN
 F 1 "+5V" H 14100 6390 30  0000 C CNN
 F 2 "" H 14100 6300 60  0001 C CNN
@@
 $EndComp
 $Comp
-L PWR_FLAG #FLG?
+L PWR_FLAG #FLG3
 U 1 1 5813F81B
 P 14300 6300
-F 0 "#FLG?" H 14300 6395 30  0001 C CNN
+F 0 "#FLG3" H 14300 6395 30  0001 C CNN
 F 1 "PWR_FLAG" H 14300 6480 30  0000 C CNN
 F 2 "" H 14300 6300 60  0001 C CNN
@@
 SYS_5V: Low-current supply\nprovided by BeagleBone PMIC\nActive when BeagleBone is running
 $Comp
-L +3.3V #PWR?
+L +3.3V #PWR2
 U 1 1 5813F81C
 P 14100 5900
-F 0 "#PWR?" H 14100 5860 30  0001 C CNN
+F 0 "#PWR2" H 14100 5860 30  0001 C CNN
 F 1 "+3.3V" H 14100 6010 30  0000 C CNN
 F 2 "" H 14100 5900 60  0001 C CNN
@@
 NoConn ~ 14350 8800
 $Comp
-L GND #PWR?
+L GND #PWR4
 U 1 1 5813F81D
 P 14500 8400
-F 0 "#PWR?" H 14500 8400 30  0001 C CNN
+F 0 "#PWR4" H 14500 8400 30  0001 C CNN
 F 1 "GND" H 14500 8330 30  0001 C CNN
 F 2 "" H 14500 8400 60  0001 C CNN
@@
 	1    0    0    -1
 $EndComp
-Text GLabel 5100 4800 0    50   UnSpc ~ 0
+Text GLabel 4800 4800 0    50   UnSpc ~ 0
 D3.3V
 Text GLabel 6050 4800 2    50   UnSpc ~ 0
@@
 Text GLabel 5550 4300 0    50   Output ~ 0
 STEP_W
-Text GLabel 5100 4700 0    50   UnSpc ~ 0
+Text GLabel 4800 4700 0    50   UnSpc ~ 0
 ADC_VDD
 Text GLabel 6050 5950 2    50   UnSpc ~ 0
@@
 ESTOP
 $Comp
-L CONN_02X05 ADC
+L CONN_02X05 ADC1
 U 1 1 58141E82
 P 5800 5750
-F 0 "ADC" H 5800 6050 50  0000 C CNN
+F 0 "ADC1" H 5800 6050 50  0000 C CNN
 F 1 "CONN_02X05" H 5800 5450 50  0000 C CNN
 F 2 "" H 5800 4550 50  0000 C CNN
@@
 DGND
 Wire Wire Line
-	5100 4700 5150 4700
-Wire Wire Line
-	5150 4700 5150 4800
-Connection ~ 5150 4800
-Wire Wire Line
-	5550 4800 5100 4800
+	4800 4700 4900 4700
+Wire Wire Line
+	4900 4700 4900 5500
+Connection ~ 4900 4800
+Wire Wire Line
+	4800 4800 5550 4800
 Text GLabel 8700 4350 2    50   Output ~ 0
 SDA
 Text GLabel 5550 5100 0    50   Input ~ 0
 SDA
+$Comp
+L R R1
+U 1 1 599361DE
+P 4900 5650
+F 0 "R1" V 4980 5650 50  0000 C CNN
+F 1 "120R" V 4900 5650 50  0000 C CNN
+F 2 "" V 4830 5650 50  0000 C CNN
+F 3 "" H 4900 5650 50  0000 C CNN
+	1    4900 5650
+	1    0    0    -1
+$EndComp
+Wire Wire Line
+	4900 5800 4900 5950
+Wire Wire Line
+	4900 5950 5550 5950
 $EndSCHEMATC

Commit message: Add version 2
Signed-off-by: Michael Brown <producer@holotronic.dk>
Parts:
- removed GPIO_1: CONN_02X20, symbol CONN_02X20
- removed P1: SOCKET_6_LONG, pin_strip_6, symbol HEADER_6
- added R2: 120R, Resistor_SMD:R_1206_3216Metric_Pad1.42x1.75mm_HandSolder, symbol Cramps2_nano-soc-rescue:R
- ADC1: footprint (none) -> Connector_PinHeader_2.54mm:PinHeader_2x05_P2.54mm_Horizontal; symbol CONN_02X05 -> Cramps2_nano-soc-rescue:CONN_02X05
- GPIO_0: footprint (none) -> Connector_PinHeader_2.54mm:PinHeader_2x20_P2.54mm_Vertical; symbol CONN_02X20 -> Cramps2_nano-soc-rescue:CONN_02X20
- P8: footprint P8P9_PinHeader -> Connector_PinHeader_2.54mm:PinHeader_2x23_P2.54mm_Vertical; symbol BB_EXP_CONN_P8 -> Cramps2_nano-soc-rescue:BB_EXP_CONN_P8
- P9: footprint P8P9_PinHeader -> Connector_PinHeader_2.54mm:PinHeader_2x23_P2.54mm_Vertical; symbol BB_EXP_CONN_P9 -> Cramps2_nano-soc-rescue:BB_EXP_CONN_P9
- R1: footprint (none) -> Resistor_THT:R_Axial_DIN0207_L6.3mm_D2.5mm_P7.62mm_Horizontal; symbol R -> Cramps2_nano-soc-rescue:R
Connections:
- net VDD_5V is gone; now on net +5V: GPIO_0.11 (P11), P9.5 (VDD_5V), P9.6 (VDD_5V)
- net +3V3: now also R2.1
- net at ADC1.9 (P9), R1.2: now also R2.2
- net PWR_BUT: no longer names the net of P9.9 (PWR_BUT)
- net RESETn: no longer names the net of P9.10 (SYS_RESETn)
- no-connect marks 35 -> 30
Other:
- note added: "or"
- note removed: "BeagleBone serial\nconsole pass-through\nheader"
- note removed: "Serial\nConsole"
- note removed: "Uses Arduino 6-pin\nstacking connector\nfor low-cost"
Changed lines of the file:
@@
-EESchema Schematic File Version 2
-LIBS:power
-LIBS:device
-LIBS:transistors
-LIBS:conn
-LIBS:linear
-LIBS:regul
-LIBS:74xx
-LIBS:cmos4000
-LIBS:adc-dac
-LIBS:memory
-LIBS:xilinx
-LIBS:microcontrollers
-LIBS:dsp
-LIBS:microchip
-LIBS:analog_switches
-LIBS:motorola
-LIBS:texas
-LIBS:intel
-LIBS:audio
-LIBS:interface
-LIBS:digital-audio
-LIBS:philips
-LIBS:display
-LIBS:cypress
-LIBS:siliconi
-LIBS:opto
-LIBS:atmel
-LIBS:contrib
-LIBS:valves
+EESchema Schematic File Version 4
 LIBS:Cramps2_nano-soc-cache
-EELAYER 25 0
+EELAYER 26 0
 EELAYER END
 $Descr A3 16535 11693
@@
 Text GLabel 7500 3550 0    50   UnSpc ~ 0
 D3.3V
-Text GLabel 8700 3850 2    50   Output ~ 0
-RESETn
-Text GLabel 7500 3850 0    50   Output ~ 0
-PWR_BUT
 Text GLabel 7500 4450 0    50   Input ~ 0
 FET4
@@
 Text GLabel 8700 5050 2    50   UnSpc ~ 0
 ADC_GND
-Text Notes 14700 8300 0    50   ~ 0
-BeagleBone serial\nconsole pass-through\nheader
 Text GLabel 8700 3450 2    50   UnSpc ~ 0
 DGND
@@
 DGND
 $Comp
-L PWR_FLAG #FLG1
+L power:PWR_FLAG #FLG01
 U 1 1 5813F80B
 P 14050 6850
-F 0 "#FLG1" H 14050 6945 30  0001 C CNN
+F 0 "#FLG01" H 14050 6945 30  0001 C CNN
 F 1 "PWR_FLAG" H 14050 7030 30  0000 C CNN
 F 2 "" H 14050 6850 60  0001 C CNN
@@
 $EndComp
 $Comp
-L GND #PWR1
+L power:GND #PWR01
 U 1 1 5813F80C
 P 14050 6950
-F 0 "#PWR1" H 14050 6950 30  0001 C CNN
+F 0 "#PWR01" H 14050 6950 30  0001 C CNN
 F 1 "GND" H 14050 6880 30  0001 C CNN
 F 2 "" H 14050 6950 60  0001 C CNN
@@
 	14050 6850 14050 6950
 $Comp
-L BB_EXP_CONN_P8 P8
+L Cramps2_nano-soc-rescue:BB_EXP_CONN_P8 P8
 U 1 1 5813F816
 P 8100 7100
 F 0 "P8" H 8095 8355 60  0000 C CNN
 F 1 "BB_EXP_CONN" H 8100 5885 60  0001 C CNN
-F 2 "P8P9_PinHeader" H 7750 5900 60  0001 C CNN
+F 2 "Connector_PinHeader_2.54mm:PinHeader_2x23_P2.54mm_Vertical" H 7750 5900 60  0001 C CNN
 F 3 "" H 7750 5900 60  0000 C CNN
 F 4 "Major League" H 8100 7100 60  0001 C CNN "Mfg"
@@
 $EndComp
 $Comp
-L BB_EXP_CONN_P9 P9
+L Cramps2_nano-soc-rescue:BB_EXP_CONN_P9 P9
 U 1 1 5813F817
 P 8100 4550
 F 0 "P9" H 8095 5805 60  0000 C CNN
 F 1 "BB_EXP_CONN" H 8100 3330 60  0001 C CNN
-F 2 "P8P9_PinHeader" H 7750 3350 60  0001 C CNN
+F 2 "Connector_PinHeader_2.54mm:PinHeader_2x23_P2.54mm_Vertical" H 7750 3350 60  0001 C CNN
 F 3 "" H 7750 3350 60  0000 C CNN
 F 4 "Major League" H 8100 1750 60  0001 C CNN "Mfg"
@@
 	1    0    0    -1
 $EndComp
-$Comp
-L HEADER_6 P1
-U 1 1 5813F818
-P 14250 8550
-F 0 "P1" H 14250 8900 60  0000 C CNN
-F 1 "SOCKET_6_LONG" H 14250 8200 60  0001 C CNN
-F 2 "pin_strip_6" H 14250 8550 60  0001 C CNN
-F 3 "" H 14250 8550 60  0000 C CNN
-F 4 "Sparkfun" H 14250 8550 60  0001 C CNN "Mfg"
-F 5 "PRT-09280" H 14250 8550 60  0001 C CNN "PartNo"
-	1    14250 8550
-	-1   0    0    -1
-$EndComp
-Wire Wire Line
-	13850 6000 14300 6000
-Wire Wire Line
-	13850 6400 14300 6400
+Wire Wire Line
+	13850 6000 14100 6000
+Wire Wire Line
+	13850 6400 14100 6400
 Text GLabel 13850 6000 0    50   UnSpc ~ 0
 D3.3V
@@
 BeagleBone Logic supply is always 3.3V
 $Comp
-L PWR_FLAG #FLG2
+L power:PWR_FLAG #FLG02
 U 1 1 5813F819
 P 14300 5900
-F 0 "#FLG2" H 14300 5995 30  0001 C CNN
+F 0 "#FLG02" H 14300 5995 30  0001 C CNN
 F 1 "PWR_FLAG" H 14300 6080 30  0000 C CNN
 F 2 "" H 14300 5900 60  0001 C CNN
@@
 	14100 6400 14100 6300
 $Comp
-L +5V #PWR3
+L power:+5V #PWR03
 U 1 1 5813F81A
 P 14100 6300
-F 0 "#PWR3" H 14100 6390 20  0001 C CNN
+F 0 "#PWR03" H 14100 6390 20  0001 C CNN
 F 1 "+5V" H 14100 6390 30  0000 C CNN
 F 2 "" H 14100 6300 60  0001 C CNN
@@
 $EndComp
 $Comp
-L PWR_FLAG #FLG3
+L power:PWR_FLAG #FLG03
 U 1 1 5813F81B
 P 14300 6300
-F 0 "#FLG3" H 14300 6395 30  0001 C CNN
+F 0 "#FLG03" H 14300 6395 30  0001 C CNN
 F 1 "PWR_FLAG" H 14300 6480 30  0000 C CNN
 F 2 "" H 14300 6300 60  0001 C CNN
@@
 SYS_5V: Low-current supply\nprovided by BeagleBone PMIC\nActive when BeagleBone is running
 $Comp
-L +3.3V #PWR2
+L power:+3.3V #PWR02
 U 1 1 5813F81C
 P 14100 5900
-F 0 "#PWR2" H 14100 5860 30  0001 C CNN
+F 0 "#PWR02" H 14100 5860 30  0001 C CNN
 F 1 "+3.3V" H 14100 6010 30  0000 C CNN
 F 2 "" H 14100 5900 60  0001 C CNN
@@
 Wire Wire Line
 	14300 6000 14300 5900
-NoConn ~ 14350 8400
-NoConn ~ 14350 8500
-NoConn ~ 14350 8600
-NoConn ~ 14350 8700
-NoConn ~ 14350 8800
-$Comp
-L GND #PWR4
-U 1 1 5813F81D
-P 14500 8400
-F 0 "#PWR4" H 14500 8400 30  0001 C CNN
-F 1 "GND" H 14500 8330 30  0001 C CNN
-F 2 "" H 14500 8400 60  0001 C CNN
-F 3 "" H 14500 8400 60  0001 C CNN
-	1    14500 8400
-	1    0    0    -1
-$EndComp
-Wire Wire Line
-	14350 8300 14500 8300
-Wire Wire Line
-	14500 8300 14500 8400
 Text Notes 14600 6000 0    50   ~ 0
 D3.3V: Low-current supply\nfrom 500 mA LDO on BeagleBone
 Text GLabel 8700 6700 2    50   Input ~ 0
 DIR_U
-Text Notes 14000 7900 0    100  ~ 0
-Serial\nConsole
-Text Notes 14700 8600 0    50   ~ 0
-Uses Arduino 6-pin\nstacking connector\nfor low-cost
-$Comp
-L CONN_02X20 GPIO_0
+$Comp
+L Cramps2_nano-soc-rescue:CONN_02X20 GPIO_0
 U 1 1 581404F4
 P 5800 4350
 F 0 "GPIO_0" H 5800 5400 50  0000 C CNN
 F 1 "CONN_02X20" V 5800 4350 50  0000 C CNN
-F 2 "" H 5800 3400 50  0000 C CNN
+F 2 "Connector_PinHeader_2.54mm:PinHeader_2x20_P2.54mm_Vertical" H 5800 3400 50  0001 C CNN
 F 3 "" H 5800 3400 50  0000 C CNN
 	1    5800 4350
@@
 Text GLabel 5550 4300 0    50   Output ~ 0
 STEP_W
-Text GLabel 4800 4700 0    50   UnSpc ~ 0
-ADC_VDD
 Text GLabel 6050 5950 2    50   UnSpc ~ 0
 ADC_GND
-$Comp
-L CONN_02X20 GPIO_1
-U 1 1 58141668
-P 5800 7250
-F 0 "GPIO_1" H 5800 8300 50  0000 C CNN
-F 1 "CONN_02X20" V 5800 7250 50  0000 C CNN
-F 2 "" H 5800 6300 50  0000 C CNN
-F 3 "" H 5800 6300 50  0000 C CNN
-	1    5800 7250
-	1    0    0    -1
-$EndComp
 Text GLabel 5550 4400 0    50   Output ~ 0
 FET1
@@
 ESTOP
 $Comp
-L CONN_02X05 ADC1
+L Cramps2_nano-soc-rescue:CONN_02X05 ADC1
 U 1 1 58141E82
 P 5800 5750
 F 0 "ADC1" H 5800 6050 50  0000 C CNN
 F 1 "CONN_02X05" H 5800 5450 50  0000 C CNN
-F 2 "" H 5800 4550 50  0000 C CNN
+F 2 "Connector_PinHeader_2.54mm:PinHeader_2x05_P2.54mm_Horizontal" H 5800 4550 50  0001 C CNN
 F 3 "" H 5800 4550 50  0000 C CNN
 	1    5800 5750
@@
 Text GLabel 6050 3900 2    50   UnSpc ~ 0
 DGND
-Wire Wire Line
-	4800 4700 4900 4700
-Wire Wire Line
-	4900 4700 4900 5500
 Connection ~ 4900 4800
 Wire Wire Line
-	4800 4800 5550 4800
+	4800 4800 4900 4800
 Text GLabel 8700 4350 2    50   Output ~ 0
 SDA
@@
 SDA
 $Comp
-L R R1
+L Cramps2_nano-soc-rescue:R R1
 U 1 1 599361DE
 P 4900 5650
 F 0 "R1" V 4980 5650 50  0000 C CNN
 F 1 "120R" V 4900 5650 50  0000 C CNN
-F 2 "" V 4830 5650 50  0000 C CNN
+F 2 "Resistor_THT:R_Axial_DIN0207_L6.3mm_D2.5mm_P7.62mm_Horizontal" V 4830 5650 50  0001 C CNN
 F 3 "" H 4900 5650 50  0000 C CNN
 	1    4900 5650
@@
 Wire Wire Line
 	4900 5950 5550 5950
+Wire Wire Line
+	14100 6400 14300 6400
+Wire Wire Line
+	14100 6000 14300 6000
+Wire Wire Line
+	4900 4800 4900 5500
+Wire Wire Line
+	4900 4800 5550 4800
+Wire Wire Line
+	4900 4700 4900 4800
+Wire Wire Line
+	4800 4700 4900 4700
+Text GLabel 4800 4700 0    50   UnSpc ~ 0
+ADC_VDD
+Text GLabel 13850 6550 0    50   UnSpc ~ 0
+VDD_5V
+Wire Wire Line
+	13850 6550 14100 6550
+Wire Wire Line
+	14100 6550 14100 6400
+$Comp
+L Cramps2_nano-soc-rescue:R R2
+U 1 1 5CB8CE43
+P 4620 5650
+F 0 "R2" V 4700 5650 50  0000 C CNN
+F 1 "120R" V 4620 5650 50  0000 C CNN
+F 2 "Resistor_SMD:R_1206_3216Metric_Pad1.42x1.75mm_HandSolder" V 4550 5650 50  0001 C CNN
+F 3 "" H 4620 5650 50  0000 C CNN
+	1    4620 5650
+	1    0    0    -1
+$EndComp
+Wire Wire Line
+	4620 5500 4900 5500
+Connection ~ 4900 5500
+Wire Wire Line
+	4620 5800 4900 5800
+Connection ~ 4900 5800
+Text Notes 4740 5680 0    60   ~ 0
+or
 $EndSCHEMATC
